Commit message: starting to add cube + 3 cameras

File: so100.urdf (robot description, URDF)
Before this commit: robot so_arm100, 7 links, 6 joints
Links:
- added link side_camera, mass 0.05; collision box size=0.03 0.03 0.02; visual box size=0.03 0.03 0.02
- added link top_camera, mass 0.05; collision box size=0.03 0.03 0.02; visual box size=0.03 0.03 0.02
- added link wrist_camera, mass 0.01; collision box size=0.02 0.02 0.01; visual box size=0.02 0.02 0.01
Joints:
- added joint side_camera_joint: type fixed, parent base, child side_camera, origin xyz=0.6 0 0.3 rpy=0 0 -1.57079
- added joint top_camera_joint: type fixed, parent base, child top_camera, origin xyz=0 0.3 0.8 rpy=0 1.57079 0
- added joint wrist_camera_joint: type fixed, parent wrist, child wrist_camera, origin xyz=0 -0.08 0.02 rpy=0 0 0
- joint shoulder_pan: limit lower=-2 upper=2 effort=35 velocity=1 -> lower=-1.57079 upper=1.57079 effort=35 velocity=1

Commit message: wrist camera position calibration

File: so100.urdf (robot description, URDF)
Before this commit: robot so_arm100, 10 links, 9 joints
Joints:
- joint wrist_camera_joint: origin xyz=0 -0.08 0.02 rpy=0 0 0 -> xyz=-0.660 0.070 1.270 rpy=0.0000 0.6109 -2.0944
- joint wrist_roll: origin xyz=0 -0.0601 0 rpy=0 1.57079 0 -> xyz=0 -0.0601 0 rpy=0 3.14159 0

Commit message: wrist camera rotation

File: so100.urdf (robot description, URDF)
Before this commit: robot so_arm100, 10 links, 9 joints
Links:
- link wrist_camera: geometry collision box size=0.05 0.05 0.03; visual box size=0.05 0.05 0.03
Joints:
- joint wrist_camera_joint: origin xyz=-0.660 0.070 1.270 rpy=0.0000 0.6109 -2.0944 -> xyz=0.0 -0.075 0 rpy=0.0 0.0 0.0

Commit message: wrist camera rotate wip

File: so100.urdf (robot description, URDF)
Before this commit: robot so_arm100, 10 links, 9 joints
Joints:
- joint wrist_camera_joint: origin xyz=0.0 -0.075 0 rpy=0.0 0.0 0.0 -> xyz=0.0 -0.05 0.20 rpy=0.0 -1.57079 0.0

Commit message: rotation now works, tho wrist camera angle is off

File: so100.urdf (robot description, URDF)
Before this commit: robot so_arm100, 10 links, 9 joints
Joints:
- joint wrist_camera_joint: origin xyz=0.0 -0.05 0.20 rpy=0.0 -1.57079 0.0 -> xyz=0.0 -0.12 0.15 rpy=0.0 -1.57079 0.0

Commit message: finished wrist camera

File: so100.urdf (robot description, URDF)
Before this commit: robot so_arm100, 10 links, 9 joints
Joints:
- joint wrist_camera_joint: origin xyz=0.0 -0.12 0.15 rpy=0.0 -1.57079 0.0 -> xyz=0 0 0 rpy=0 -1.57079 0

Commit message: heuristic policy positioning adjusted. reward needs work, grasp not registering.

File: so100.urdf (robot description, URDF)
Before this commit: robot so_arm100, 10 links, 9 joints
Links:
- link gripper: geometry collision mesh filename=assets/Fixed_Jaw.stl; visual mesh filename=assets/Fixed_Jaw.stl
- link jaw: geometry collision mesh filename=assets/Moving_Jaw.stl; visual mesh filename=assets/Moving_Jaw.stl

Commit message: replaced rmpflow with pure kinematics

File: so100.urdf (robot description, URDF)
Before this commit: robot so_arm100, 7 links, 6 joints
Links:
- link base: geometry collision mesh filename=assets/Base.stl scale=0.001 0.001 0.001; visual mesh filename=assets/Base.stl scale=0.001 0.001 0.001
- link gripper: geometry collision mesh filename=assets/Fixed_Jaw.stl scale=0.001 0.001 0.001; visual mesh filename=assets/Fixed_Jaw.stl scale=0.001 0.001 0.001
- link jaw: geometry collision mesh filename=assets/Moving_Jaw.stl scale=0.001 0.001 0.001; visual mesh filename=assets/Moving_Jaw.stl scale=0.001 0.001 0.001
- link lower_arm: geometry collision mesh filename=assets/Lower_Arm.stl scale=0.001 0.001 0.001; visual mesh filename=assets/Lower_Arm.stl scale=0.001 0.001 0.001
- link shoulder: geometry collision mesh filename=assets/Rotation_Pitch.stl scale=0.001 0.001 0.001; visual mesh filename=assets/Rotation_Pitch.stl scale=0.001 0.001 0.001
- link upper_arm: geometry collision mesh filename=assets/Upper_Arm.stl scale=0.001 0.001 0.001; visual mesh filename=assets/Upper_Arm.stl scale=0.001 0.001 0.001
- link wrist: geometry collision mesh filename=assets/Wrist_Pitch_Roll.stl scale=0.001 0.001 0.001; visual mesh filename=assets/Wrist_Pitch_Roll.stl scale=0.001 0.001 0.001
Joints:
- joint elbow_flex: origin xyz=0 0.281425 0.07 rpy=1.57079 0 0 -> xyz=0 0 0.117 rpy=0 0 0
- joint shoulder_lift: limit lower=0 upper=3.5 effort=35 velocity=1 -> lower=-1.57079 upper=1.57079 effort=35 velocity=1; origin xyz=0 0.25625 0.0765 rpy=-1.8 0 0 -> xyz=0 0 0 rpy=0 0 0
- joint shoulder_pan: axis 0 1 0 -> 0 0 1; origin xyz=0 -0.113 0.04125 rpy=1.57079 0 0 -> xyz=0 0 0.120 rpy=0 0 0
- joint wrist_flex: limit lower=-2.5 upper=1.2 effort=35 velocity=1 -> lower=-1.745 upper=1.745 effort=35 velocity=1; origin xyz=0 0.013 0.33725 rpy=-1 0 0 -> xyz=0 0 0.136 rpy=0 0 0
- joint wrist_roll: axis 0 1 0 -> 0 0 1; origin xyz=0 -0.15025 0 rpy=0 3.14159 0 -> xyz=0 0 0 rpy=0 0 0

Commit message: replaced rmpflow with pure kinematics

File: so100.urdf (robot description, URDF)
Before this commit: robot so_arm100, 7 links, 6 joints
Links:
- link base: geometry collision mesh filename=assets/Base.stl scale=1.0 1.0 1.0; visual mesh filename=assets/Base.stl scale=1.0 1.0 1.0
- link gripper: geometry collision mesh filename=assets/Fixed_Jaw.stl scale=1.0 1.0 1.0; visual mesh filename=assets/Fixed_Jaw.stl scale=1.0 1.0 1.0
- link jaw: geometry collision mesh filename=assets/Moving_Jaw.stl scale=1.0 1.0 1.0; visual mesh filename=assets/Moving_Jaw.stl scale=1.0 1.0 1.0
- link lower_arm: geometry collision mesh filename=assets/Lower_Arm.stl scale=1.0 1.0 1.0; visual mesh filename=assets/Lower_Arm.stl scale=1.0 1.0 1.0
- link shoulder: geometry collision mesh filename=assets/Rotation_Pitch.stl scale=1.0 1.0 1.0; visual mesh filename=assets/Rotation_Pitch.stl scale=1.0 1.0 1.0
- link upper_arm: geometry collision mesh filename=assets/Upper_Arm.stl scale=1.0 1.0 1.0; visual mesh filename=assets/Upper_Arm.stl scale=1.0 1.0 1.0
- link wrist: geometry collision mesh filename=assets/Wrist_Pitch_Roll.stl scale=1.0 1.0 1.0; visual mesh filename=assets/Wrist_Pitch_Roll.stl scale=1.0 1.0 1.0

Commit message: replaced rmpflow with pure kinematics

File: so100.urdf (robot description, URDF)
Before this commit: robot so_arm100, 7 links, 6 joints
Joints:
- joint elbow_flex: origin xyz=0 0 0.117 rpy=0 0 0 -> xyz=0 0.11257 0.028 rpy=1.57079 0 0
- joint shoulder_lift: limit lower=-1.57079 upper=1.57079 effort=35 velocity=1 -> lower=0 upper=3.5 effort=35 velocity=1; origin xyz=0 0 0 rpy=0 0 0 -> xyz=0 0.1025 0.0306 rpy=-1.8 0 0
- joint shoulder_pan: axis 0 0 1 -> 0 1 0; origin xyz=0 0 0.120 rpy=0 0 0 -> xyz=0 -0.0452 0.0165 rpy=1.57079 0 0
- joint wrist_flex: limit lower=-1.745 upper=1.745 effort=35 velocity=1 -> lower=-2.5 upper=1.2 effort=35 velocity=1; origin xyz=0 0 0.136 rpy=0 0 0 -> xyz=0 0.0052 0.1349 rpy=-1 0 0
- joint wrist_roll: axis 0 0 1 -> 0 1 0; origin xyz=0 0 0 rpy=0 0 0 -> xyz=0 -0.0601 0 rpy=0 3.14159 0

Commit message: replaced rmpflow with pure kinematics

File: so100.urdf (robot description, URDF)
Before this commit: robot so_arm100, 7 links, 6 joints
Joints:
- joint gripper: origin xyz=-0.0505 -0.061 0 rpy=0 3.14158 0 -> xyz=-0.0202 -0.0244 0 rpy=0 3.14158 0

Commit message: replaced rmpflow with pure kinematics

File: so100.urdf (robot description, URDF)
Before this commit: robot so_arm100, 7 links, 6 joints
Links:
- link base: geometry collision mesh filename=assets/Base.stl scale=0.001 0.001 0.001; visual mesh filename=assets/Base.stl scale=0.001 0.001 0.001
- link gripper: geometry collision mesh filename=assets/Fixed_Jaw.stl scale=0.001 0.001 0.001; visual mesh filename=assets/Fixed_Jaw.stl scale=0.001 0.001 0.001
- link jaw: geometry collision mesh filename=assets/Moving_Jaw.stl scale=0.001 0.001 0.001; visual mesh filename=assets/Moving_Jaw.stl scale=0.001 0.001 0.001
- link lower_arm: geometry collision mesh filename=assets/Lower_Arm.stl scale=0.001 0.001 0.001; visual mesh filename=assets/Lower_Arm.stl scale=0.001 0.001 0.001
- link shoulder: geometry collision mesh filename=assets/Rotation_Pitch.stl scale=0.001 0.001 0.001; visual mesh filename=assets/Rotation_Pitch.stl scale=0.001 0.001 0.001
- link upper_arm: geometry collision mesh filename=assets/Upper_Arm.stl scale=0.001 0.001 0.001; visual mesh filename=assets/Upper_Arm.stl scale=0.001 0.001 0.001
- link wrist: geometry collision mesh filename=assets/Wrist_Pitch_Roll.stl scale=0.001 0.001 0.001; visual mesh filename=assets/Wrist_Pitch_Roll.stl scale=0.001 0.001 0.001
Joints:
- joint elbow_flex: origin xyz=0 0.11257 0.028 rpy=1.57079 0 0 -> xyz=0 0.1135 0.0282 rpy=1.57079 0 0
- joint shoulder_lift: origin xyz=0 0.1025 0.0306 rpy=-1.8 0 0 -> xyz=0 0.1025 0.10125 rpy=-1.8 0 0
- joint shoulder_pan: origin xyz=0 -0.0452 0.0165 rpy=1.57079 0 0 -> xyz=0 -0.0452 0.01875 rpy=1.57079 0 0
- joint wrist_flex: origin xyz=0 0.0052 0.1349 rpy=-1 0 0 -> xyz=0 0.0052 0.1359 rpy=-1 0 0

Commit message: replaced rmpflow with pure kinematics

File: so100.urdf (robot description, URDF)
Before this commit: robot so_arm100, 7 links, 6 joints
Joints:
- joint elbow_flex: origin xyz=0 0.1135 0.0282 rpy=1.57079 0 0 -> xyz=0 0.11257 0.028 rpy=1.57079 0 0
- joint shoulder_lift: origin xyz=0 0.1025 0.10125 rpy=-1.8 0 0 -> xyz=0 0.1025 0.0306 rpy=-1.8 0 0
- joint shoulder_pan: origin xyz=0 -0.0452 0.01875 rpy=1.57079 0 0 -> xyz=0 -0.0452 0.0165 rpy=1.57079 0 0
- joint wrist_flex: origin xyz=0 0.0052 0.1359 rpy=-1 0 0 -> xyz=0 0.0052 0.1349 rpy=-1 0 0

Commit message: replaced rmpflow with pure kinematics

File: so100.urdf (robot description, URDF)
Before this commit: robot so_arm100, 7 links, 6 joints
Links:
- link base: geometry collision mesh filename=assets/Base.stl scale=1.0 1.0 1.0; visual mesh filename=assets/Base.stl scale=1.0 1.0 1.0
- link gripper: geometry collision mesh filename=assets/Fixed_Jaw.stl scale=1.0 1.0 1.0; visual mesh filename=assets/Fixed_Jaw.stl scale=1.0 1.0 1.0
- link jaw: geometry collision mesh filename=assets/Moving_Jaw.stl scale=1.0 1.0 1.0; visual mesh filename=assets/Moving_Jaw.stl scale=1.0 1.0 1.0
- link lower_arm: geometry collision mesh filename=assets/Lower_Arm.stl scale=1.0 1.0 1.0; visual mesh filename=assets/Lower_Arm.stl scale=1.0 1.0 1.0
- link shoulder: geometry collision mesh filename=assets/Rotation_Pitch.stl scale=1.0 1.0 1.0; visual mesh filename=assets/Rotation_Pitch.stl scale=1.0 1.0 1.0
- link upper_arm: geometry collision mesh filename=assets/Upper_Arm.stl scale=1.0 1.0 1.0; visual mesh filename=assets/Upper_Arm.stl scale=1.0 1.0 1.0
- link wrist: geometry collision mesh filename=assets/Wrist_Pitch_Roll.stl scale=1.0 1.0 1.0; visual mesh filename=assets/Wrist_Pitch_Roll.stl scale=1.0 1.0 1.0
Joints:
- joint elbow_flex: origin xyz=0 0.11257 0.028 rpy=1.57079 0 0 -> xyz=0 0.1135 0.028 rpy=1.57079 0 0
- joint shoulder_pan: origin xyz=0 -0.0452 0.0165 rpy=1.57079 0 0 -> xyz=0 -0.0452 0.0435 rpy=1.57079 0 0
- joint wrist_flex: origin xyz=0 0.0052 0.1349 rpy=-1 0 0 -> xyz=0 0.0052 0.1359 rpy=-1 0 0

Commit message: adjust shoulder link

File: so100.urdf (robot description, URDF)
Before this commit: robot so_arm100, 7 links, 6 joints
Joints:
- joint shoulder_pan: origin xyz=0 -0.0452 0.0435 rpy=1.57079 0 0 -> xyz=0 -0.0452 0.0165 rpy=1.57079 0 0

Commit message: penalize self-collision

File: so100.urdf (robot description, URDF)
Before this commit: robot so_arm100, 7 links, 6 joints
Links:
- link base: geometry collision cylinder length=0.05 radius=0.04; visual mesh filename=assets/Base.stl scale=1.0 1.0 1.0
- link gripper: geometry collision box size=0.04 0.05 0.03; visual mesh filename=assets/Fixed_Jaw.stl scale=1.0 1.0 1.0
- link jaw: geometry collision box size=0.02 0.04 0.02; visual mesh filename=assets/Moving_Jaw.stl scale=1.0 1.0 1.0
- link lower_arm: geometry collision box size=0.04 0.04 0.14; visual mesh filename=assets/Lower_Arm.stl scale=1.0 1.0 1.0
- link shoulder: geometry collision box size=0.05 0.08 0.05; visual mesh filename=assets/Rotation_Pitch.stl scale=1.0 1.0 1.0
- link upper_arm: geometry collision box size=0.04 0.12 0.04; visual mesh filename=assets/Upper_Arm.stl scale=1.0 1.0 1.0
- link wrist: geometry collision box size=0.04 0.06 0.04; visual mesh filename=assets/Wrist_Pitch_Roll.stl scale=1.0 1.0 1.0

Commit message: reached debug

File: so100.urdf (robot description, URDF)
Before this commit: robot so_arm100, 7 links, 6 joints
Links:
- link gripper: geometry collision box size=0.05 0.07 0.04; visual mesh filename=assets/Fixed_Jaw.stl scale=1.0 1.0 1.0
- link jaw: geometry collision box size=0.03 0.06 0.03; visual mesh filename=assets/Moving_Jaw.stl scale=1.0 1.0 1.0

Commit message: mesh collider gripper

File: so100.urdf (robot description, URDF)
Before this commit: robot so_arm100, 7 links, 6 joints
Links:
- link gripper: geometry collision mesh filename=assets/Fixed_Jaw.stl scale=1.0 1.0 1.0; visual mesh filename=assets/Fixed_Jaw.stl scale=1.0 1.0 1.0
- link jaw: geometry collision mesh filename=assets/Moving_Jaw.stl scale=1.0 1.0 1.0; visual mesh filename=assets/Moving_Jaw.stl scale=1.0 1.0 1.0

Commit message: stop gripper clipping into cube

File: so100.urdf (robot description, URDF)
Before this commit: robot so_arm100, 7 links, 6 joints
Links:
- link gripper: geometry collision box size=0.015 0.05 0.025; visual mesh filename=assets/Fixed_Jaw.stl scale=1.0 1.0 1.0
- link jaw: geometry collision box size=0.015 0.05 0.025; visual mesh filename=assets/Moving_Jaw.stl scale=1.0 1.0 1.0

Commit message: stop gripper clipping into cube

File: so100.urdf (robot description, URDF)
Before this commit: robot so_arm100, 7 links, 6 joints
Links:
- link gripper: geometry collision box size=0.015 0.05 0.025; visual box size=0.015 0.05 0.025
- link jaw: geometry collision box size=0.015 0.05 0.025; visual box size=0.015 0.05 0.025

Commit message: stop gripper clipping into cube

File: so100.urdf (robot description, URDF)
Before this commit: robot so_arm100, 7 links, 6 joints
Links:
- link gripper: geometry collision box size=0.015 0.07 0.025; visual box size=0.015 0.07 0.025
- link jaw: geometry collision box size=0.015 0.07 0.025; visual box size=0.015 0.07 0.025

Commit message: stop gripper clipping into cube

File: so100.urdf (robot description, URDF)
Before this commit: robot so_arm100, 7 links, 6 joints
Links:
- link gripper: geometry collision box size=0.015 0.09 0.025; visual box size=0.015 0.09 0.025
- link jaw: geometry collision box size=0.015 0.09 0.025; visual box size=0.015 0.09 0.025

Commit message: stop gripper clipping into cube

File: so100.urdf (robot description, URDF)
Before this commit: robot so_arm100, 7 links, 6 joints
Links:
- link jaw: geometry collision box size=0.015 0.07 0.025; visual box size=0.015 0.07 0.025

Commit message: stop gripper clipping into cube

File: so100.urdf (robot description, URDF)
Before this commit: robot so_arm100, 7 links, 6 joints
Links:
- link jaw: geometry collision box size=0.015 0.08 0.025; visual box size=0.015 0.08 0.025

Commit message: stop gripper clipping into cube

File: so100.urdf (robot description, URDF)
Before this commit: robot so_arm100, 7 links, 6 joints
Links:
- link jaw: geometry collision box size=0.015 0.075 0.025; visual box size=0.015 0.075 0.025

Commit message: stop gripper clipping into cube

File: so100.urdf (robot description, URDF)
Before this commit: robot so_arm100, 7 links, 6 joints
Links:
- link gripper: geometry collision box size=0.015 0.10 0.025; visual box size=0.015 0.10 0.025

Commit message: stop gripper clipping into cube

File: so100.urdf (robot description, URDF)
Before this commit: robot so_arm100, 7 links, 6 joints
Joints:
- joint gripper: limit lower=-0.2 upper=2.0 effort=35 velocity=1 -> lower=-0.2 upper=2.0 effort=400 velocity=1

Commit message: stop gripper clipping into cube

File: so100.urdf (robot description, URDF)
Before this commit: robot so_arm100, 7 links, 6 joints
Links:
- link gripper: mass 0.0929859 -> 0.2; geometry collision box size=0.04 0.10 0.025; visual box size=0.04 0.10 0.025
- link jaw: mass 0.0202444 -> 0.2; geometry collision box size=0.04 0.075 0.025; visual box size=0.04 0.075 0.025

Commit message: fix grasp collision

File: so100.urdf (robot description, URDF)
Before this commit: robot so_arm100, 7 links, 6 joints
Links:
- link gripper: geometry visual mesh filename=assets/Fixed_Jaw.stl scale=1.0 1.0 1.0; visual mesh filename=assets/Fixed_Jaw_Motor.stl scale=1.0 1.0 1.0
- link jaw: geometry visual mesh filename=assets/Moving_Jaw.stl scale=1.0 1.0 1.0

Commit message: fix grasp collision

File: so100.urdf (robot description, URDF)
Before this commit: robot so_arm100, 7 links, 6 joints
Joints:
- joint gripper: limit lower=-0.2 upper=2.0 effort=400 velocity=1 -> lower=-0.2 upper=2.0 effort=20.0 velocity=1

Commit message: fix grasp collision

File: so100.urdf (robot description, URDF)
Before this commit: robot so_arm100, 7 links, 6 joints
Joints:
- joint gripper: limit lower=-0.2 upper=2.0 effort=20.0 velocity=1 -> lower=-0.2 upper=2.0 effort=200.0 velocity=1

Commit message: fix grasp collision

File: so100.urdf (robot description, URDF)
Before this commit: robot so_arm100, 7 links, 6 joints
Links:
- link base: mass 1.0 -> 5.0

Commit message: fix gripper physics instability

File: so100.urdf (robot description, URDF)
Before this commit: robot so_arm100, 7 links, 6 joints
Joints:
- joint gripper: limit lower=-0.2 upper=2.0 effort=200.0 velocity=1 -> lower=-0.2 upper=2.0 effort=2.0 velocity=1

Commit message: fix gripper physics instability

File: so100.urdf (robot description, URDF)
Before this commit: robot so_arm100, 7 links, 6 joints
Joints:
- joint gripper: limit lower=-0.2 upper=2.0 effort=2.0 velocity=1 -> lower=-0.2 upper=2.0 effort=35.0 velocity=1

Commit message: fix gripper physics instability

File: so100.urdf (robot description, URDF)
Before this commit: robot so_arm100, 7 links, 6 joints
Joints:
- joint gripper: limit lower=-0.2 upper=2.0 effort=35.0 velocity=1 -> lower=-0.2 upper=2.0 effort=5.0 velocity=1

Commit message: fix gripper physics instability

File: so100.urdf (robot description, URDF)
Before this commit: robot so_arm100, 7 links, 6 joints
Joints:
- joint gripper: limit lower=-0.2 upper=2.0 effort=5.0 velocity=1 -> lower=-0.2 upper=2.0 effort=15.0 velocity=1

Commit message: fix gripper physics instability

File: so100.urdf (robot description, URDF)
Before this commit: robot so_arm100, 7 links, 6 joints
Joints:
- joint gripper: limit lower=-0.2 upper=2.0 effort=15.0 velocity=1 -> lower=-0.2 upper=2.0 effort=25.0 velocity=1

Commit message: fix false release

File: so100.urdf (robot description, URDF)
Before this commit: robot so_arm100, 7 links, 6 joints
Joints:
- joint gripper: limit lower=-0.2 upper=2.0 effort=25.0 velocity=1 -> lower=-0.2 upper=2.0 effort=30.0 velocity=1

Commit message: fix false release

File: so100.urdf (robot description, URDF)
Before this commit: robot so_arm100, 7 links, 6 joints
Joints:
- joint gripper: limit lower=-0.2 upper=2.0 effort=30.0 velocity=1 -> lower=-0.2 upper=2.0 effort=20.0 velocity=1

Commit message: increase gripper speed

File: so100.urdf (robot description, URDF)
Before this commit: robot so_arm100, 7 links, 6 joints
Joints:
- joint gripper: limit lower=-0.2 upper=2.0 effort=20.0 velocity=1 -> lower=-0.2 upper=2.0 effort=20.0 velocity=3

Commit message: increase gripper speed

File: so100.urdf (robot description, URDF)
Before this commit: robot so_arm100, 7 links, 6 joints
Joints:
- joint gripper: limit lower=-0.2 upper=2.0 effort=20.0 velocity=3 -> lower=-0.2 upper=2.0 effort=20.0 velocity=10
